File: BlueHead.kicad_pcb (KiCad board)
At the start: 2 copper layers, 53.6 x 71.4 mm, 41 parts, among them J1 CONN_01X03, J2 CONN_01X06, J3 CONN_01X06, J4 CONN_01X08, J5 CONN_01X06, J6 CONN_01X05, J7 CONN_01X05, J8 CONN_01X05, U1 Bluepill, U2 LM7805

Commit message: Issue resolving
Parts:
- removed the G*** at (102.5, 50.2)
- removed the REF*** at (88.0, 56.5)
- removed the REF*** at (88.0, 71.2)
- removed Servo_5: CONN_01X03, Pin_Headers:Pin_Header_Straight_1x03_Pitch2.54mm
- added G***: LOGO, Hardware:EP_Logo_2, B.Cu at (80.6, 86.5)
- added J9: CONN_01X04, Pin_Headers:Pin_Header_Straight_1x04_Pitch2.54mm, F.Cu at (121.0, 56.7)
- added REF***: WEEE-Logo_4.2x6mm_SilkScreen, Symbols:WEEE-Logo_4.2x6mm_SilkScreen, F.Cu at (123.6, 43.8)
- moved G*** 51.7 mm to (102.7, 40.0)
Routing:
- net GND: track 156.0 -> 169.0 mm
- net +5V: track 101.3 -> 104.0 mm
- net SDA1: track 17.2 -> 15.2 mm
- net SCL1: track 19.0 -> 17.4 mm
Other:
- board text removed: "Main Board STM32 https://github.com/Elektropioneer"
